File: pepuinoNano.kicad_pcb (KiCad board)
At the start: 2 copper layers, 21 x 51 mm, 33 parts, among them J1 USB_C_Receptacle_USB2.0_14P, J2 Conn_01x20, J3 Conn_01x20, J4 Conn_01x03, SW1 SW_Push, U1 RP2040, U3 W25Q16JVUXIQ TR, U4 MCP1700x-330xxTT, Y1 Crystal_GND24

Commit message: update the resistor r3 and r4 from 27k to 27
Parts:
- R3, R4: value 27K -> 27
Changed lines of the file:
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@@
 			)
 		)
-		(property "Value" "27K"
+		(property "Value" "27"
 			(at 0 1.17 90)
 			(layer "F.Fab")
@@
 			)
 		)
-		(property "Value" "27K"
+		(property "Value" "27"
 			(at 0 1.17 90)
 			(layer "F.Fab")
